File: data/Franks Flightsim Boards/Controler 2_25/Controler 2_25.brd (EAGLE design)
At the start: 55 x 55 mm, 21 parts, among them IC1 3_3V, IC2 5V, J3 External, J4 FEMALE 2x3

Commit message: new PCB
Updated with new pcb for 2_25 version
Parts:
- removed U$13, U$14, U$15, U$16: (no value), SparkFun-Hardware:STAND-OFF-TIGHT
- added U$1, U$2, U$3, U$4: (no value), mechanics_v5:M2.0_SW4.0_HOLE
- J2: device SparkFun-Connectors:1X16CENTER -> SparkFun-Connectors:1X16
- moved J2 22.0 mm to (49.0, 58.0)
- flipped J3 to the bottom
Routing:
- net P19: track 45.9 -> 37.2 mm
- net P23: track 42.5 -> 34.3 mm
- net P02: track 40.9 -> 48.4 mm
- net P33: track 33.1 -> 39.9 mm
- net P35: track 23.6 -> 30.5 mm
- net P32: track 28.4 -> 35.2 mm
- net P25: track 37.9 -> 44.6 mm
- net P00: track 37.4 -> 43.5 mm
- net P34: track 20.0 -> 25.7 mm
- net P18: track 39.0 -> 33.4 mm
- net P04: track 35.2 -> 39.2 mm
- net LED: track 50.5 -> 52.8 mm, vias 0 -> 1
- net P05: track 35.8 -> 34.8 mm
- net 5V: track 101.1 -> 100.2 mm
- net N$3: track 12.4 -> 11.6 mm
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Other:
- board size 55 x 55 mm -> 60 x 60 mm
