File: data/Franks Flightsim Boards/Controler 2_25/Controler 2_25.brd (EAGLE design)
At the start: 60 x 60 mm, 21 parts, among them IC1 3_3V, IC2 5V, J3 External, J4 FEMALE 2x3

Commit message: Update dev status
Parts:
- C1: device resistor:C0805 -> resistor:C1206
- C5: device resistor:153CLV-0505 -> resistor:153CLV-0605
- moved U$10 21.7 mm to (22.5, 13.0)
- moved R1 10.4 mm to (41.1, 50.2)
- moved J1 3.66 mm to (36.7, 3.81)
- moved J4 3.66 mm to (39.2, 8.89)
- moved C5 3.60 mm to (44.5, 37.2), turned to 270 degrees
- moved IC1 1.42 mm to (40.8, 26.0)
- moved C4 1.04 mm to (51.4, 14.0)
- moved C2 0.91 mm to (50.8, 24.4)
- moved IC$1 0.84 mm to (18.9, 24.3)
- moved IC$2 0.41 mm to (37.4, 44.9)
- moved C1 0.41 mm to (52.2, 31.9)
Connections:
- net P12 renamed SRV1
- removed net P13: IC$1.26, J4.1
- removed net P15: IC$1.25, J4.2
- new net SRV2: IC$1.25, J4.1
- new net SRV3: IC$1.26, J4.2
Routing:
- net SRV2: track 0.00 -> 17.0 mm
- net SRV3: track 0.00 -> 14.8 mm
- net P15: track 14.1 -> 0.00 mm
- net P13: track 9.25 -> 0.00 mm
- net N$1: track 9.98 -> 3.72 mm
- net SRV1: track 27.9 -> 32.1 mm
- net 3_3V: track 61.7 -> 64.2 mm
- net 5V: track 100.2 -> 102.5 mm
- net CAN_R: track 20.9 -> 18.8 mm
- net P02: track 48.3 -> 47.2 mm
- net P00: track 43.5 -> 42.4 mm
- net P04: track 39.2 -> 38.2 mm
- net 12V: track 44.5 -> 45.4 mm
- net P05: track 34.8 -> 34.2 mm

Commit message: update and backup
Update
Parts:
- C3, C6: device resistor:C0805 -> resistor:C1206
- moved C2 2.03 mm to (52.8, 24.4)
- moved C3 1.48 mm to (48.2, 24.6)
- moved C6 0.45 mm to (46.9, 14.2)
Routing:
- net 12V: track 45.4 -> 33.1 mm, vias 0 -> 2
- net 3_3V: track 64.2 -> 66.2 mm
Changed lines of the file:
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@@
 <attribute name="CNAME" value="Franks FlightSim Boards"/>
 <attribute name="CPROJECT" value="Franks FlightSim Boards"/>
-<attribute name="CREVISION" value="v0.2"/>
+<attribute name="CREVISION" value="v0.3"/>
 <attribute name="DESIGNER" value="Frank van Ierland"/>
 </attributes>
@@
 <attribute name="VALUE" x="36.83" y="18.6182" size="1.27" layer="25" font="vector" ratio="10" rot="R180"/>
 </element>
-<element name="C2" library="resistor" library_urn="urn:adsk.eagle:library:348" package="CT3528" package3d_urn="urn:adsk.eagle:package:25815/1" value="47uF" x="50.8" y="24.384" smashed="yes" rot="R90">
-<attribute name="NAME" x="50.4212" y="18.962" size="1.27" layer="25" rot="R90"/>
-<attribute name="VALUE" x="52.0274" y="17.3014" size="1.27" layer="27" rot="R90"/>
+<element name="C2" library="resistor" library_urn="urn:adsk.eagle:library:348" package="CT3528" package3d_urn="urn:adsk.eagle:package:25815/1" value="47uF" x="52.832" y="24.384" smashed="yes" rot="R90">
+<attribute name="NAME" x="52.4532" y="18.962" size="1.27" layer="25" rot="R90"/>
+<attribute name="VALUE" x="54.0594" y="17.3014" size="1.27" layer="27" rot="R90"/>
 </element>
 <element name="C1" library="resistor" library_urn="urn:adsk.eagle:library:348" package="C1206" package3d_urn="urn:adsk.eagle:package:26140/1" value="100nF" x="52.2224" y="31.9024" smashed="yes">
@@
 <attribute name="VALUE" x="52.637" y="6.9382" size="1.27" layer="27" rot="R90"/>
 </element>
-<element name="C3" library="resistor" library_urn="urn:adsk.eagle:library:348" package="C0805" package3d_urn="urn:adsk.eagle:package:26137/1" value="100nF" x="46.736" y="24.9936" smashed="yes" rot="R270">
-<attribute name="NAME" x="45.1612" y="23.0124" size="1.27" layer="25" rot="R270"/>
-<attribute name="VALUE" x="46.6344" y="23.0124" size="1.27" layer="27" rot="R270"/>
+<element name="C3" library="resistor" library_urn="urn:adsk.eagle:library:348" package="C1206" package3d_urn="urn:adsk.eagle:package:26140/1" value="100nF" x="48.1584" y="24.5872" smashed="yes" rot="R270">
+<attribute name="NAME" x="46.5836" y="22.606" size="1.27" layer="25" rot="R270"/>
+<attribute name="VALUE" x="48.0568" y="22.606" size="1.27" layer="27" rot="R270"/>
 </element>
 <element name="J2" library="SparkFun-Connectors" library_urn="urn:adsk.eagle:library:513" package="1X16" package3d_urn="urn:adsk.eagle:package:38258/1" value="" x="49.05" y="58" smashed="yes" rot="MR0">
@@
 <attribute name="VALUE" x="44.7362" y="44.0246" size="1.27" layer="27" rot="R270"/>
 </element>
-<element name="C6" library="resistor" library_urn="urn:adsk.eagle:library:348" package="C0805" package3d_urn="urn:adsk.eagle:package:26137/1" value="100nF" x="47.1424" y="14.6304" smashed="yes" rot="R270">
-<attribute name="NAME" x="45.5676" y="12.6492" size="1.27" layer="25" rot="R270"/>
-<attribute name="VALUE" x="47.0408" y="12.6492" size="1.27" layer="27" rot="R270"/>
+<element name="C6" library="resistor" library_urn="urn:adsk.eagle:library:348" package="C1206" package3d_urn="urn:adsk.eagle:package:26140/1" value="100nF" x="46.9392" y="14.224" smashed="yes" rot="R270">
+<attribute name="NAME" x="45.3644" y="12.2428" size="1.27" layer="25" rot="R270"/>
+<attribute name="VALUE" x="46.8376" y="12.2428" size="1.27" layer="27" rot="R270"/>
 </element>
 <element name="U$1" library="mechanics_v5" package="M2.0_SW4.0_HOLE" value="" x="3.5" y="45" locked="yes"/>
@@
 <wire x1="44.5008" y1="34.4856" x2="44.5008" y2="31.9024" width="1.016" layer="1"/>
 <wire x1="44.5008" y1="31.9024" x2="44.5008" y2="28.448" width="1.27" layer="1"/>
-<wire x1="50.8" y1="17.8816" x2="42.545" y2="17.8816" width="1.016" layer="1"/>
-<wire x1="42.545" y1="17.8816" x2="42.4688" y2="17.9578" width="1.016" layer="1"/>
-<wire x1="53.4416" y1="19.7104" x2="53.4416" y2="27.3968" width="1.016" layer="1"/>
-<wire x1="53.4416" y1="19.7104" x2="50.8" y2="17.8816" width="1.016" layer="1"/>
-<wire x1="53.4416" y1="27.3968" x2="51.0032" y2="28.448" width="1.016" layer="1"/>
 <wire x1="44.5008" y1="31.9024" x2="50.8224" y2="31.9024" width="1.016" layer="1"/>
-<wire x1="51.0032" y1="28.448" x2="44.5008" y2="28.448" width="1.016" layer="1"/>
 <wire x1="44.5008" y1="28.448" x2="43.942" y2="28.321" width="1.016" layer="1"/>
 <wire x1="50.8224" y1="31.9024" x2="50.866" y2="35.9004" width="0.762" layer="1"/>
 <wire x1="50.866" y1="35.9004" x2="50.8" y2="35.9664" width="0.762" layer="1"/>
+<wire x1="43.942" y1="28.321" x2="46.0502" y2="28.321" width="1.27" layer="1"/>
+<wire x1="46.0502" y1="28.321" x2="46.1264" y2="28.2448" width="1.27" layer="1"/>
+<via x="46.1264" y="28.2448" extent="1-16" drill="0.35"/>
+<wire x1="46.1264" y1="28.2448" x2="46.1264" y2="18.0848" width="1.27" layer="16"/>
+<via x="46.1264" y="18.0848" extent="1-16" drill="0.35"/>
+<wire x1="46.1264" y1="18.0848" x2="42.5958" y2="18.0848" width="1.27" layer="1"/>
+<wire x1="42.5958" y1="18.0848" x2="42.4688" y2="17.9578" width="1.27" layer="1"/>
 </signal>
 <signal name="CAN_D">
@@
 <contactref element="C6" pad="1"/>
 <wire x1="51.4096" y1="15.5208" x2="50.1308" y2="15.5804" width="0.508" layer="1"/>
-<wire x1="50.1308" y1="15.5804" x2="47.1424" y2="15.5804" width="0.508" layer="1"/>
-<wire x1="47.1424" y1="15.5804" x2="42.5348" y2="15.5804" width="0.508" layer="1"/>
+<wire x1="50.1308" y1="15.5804" x2="46.9392" y2="15.624" width="0.508" layer="1"/>
+<wire x1="46.9392" y1="15.624" x2="42.5348" y2="15.5804" width="0.508" layer="1"/>
 <wire x1="42.5348" y1="15.5804" x2="42.4688" y2="15.6464" width="0.508" layer="1"/>
 <polygon width="0.2032" layer="1" thermals="no">
@@
 <vertex x="39.624" y="39.0144"/>
 </polygon>
-<wire x1="50.8" y1="25.884" x2="49.5212" y2="25.9436" width="0.508" layer="1"/>
-<wire x1="49.5212" y1="25.9436" x2="46.736" y2="25.9436" width="0.508" layer="1"/>
-<wire x1="46.736" y1="25.9436" x2="46.67" y2="26.0096" width="0.508" layer="1"/>
+<wire x1="52.832" y1="25.884" x2="49.5212" y2="25.9436" width="0.508" layer="1"/>
+<wire x1="49.5212" y1="25.9436" x2="48.1584" y2="25.9872" width="0.508" layer="1"/>
+<wire x1="48.1584" y1="25.9872" x2="46.67" y2="26.0096" width="0.508" layer="1"/>
 <wire x1="46.67" y1="26.0096" x2="43.942" y2="26.0096" width="0.508" layer="1"/>
 <wire x1="43.942" y1="26.0096" x2="42.3674" y2="26.1618" width="0.508" layer="1"/>

Commit message: backup
Parts:
- removed J1: (no value), SparkFun-Connectors:1X03
- J3: value External -> 22-27-2041-04; device con-molex:6410-05 -> con-molex:6410-04
- moved J3 1.02 mm to (50.8, 42.1)
Connections:
- removed net SRV3: IC$1.26, J4.2
- net 12V: now also J3.4; no longer J3.5
- net 3_3V: now also IC$2.3
- net 5V: no longer IC$2.3, J1.2
- net GND: now also J3.3; no longer J1.1, J3.4
- net LED: now also IC$1.2; no longer J3.3
- net SRV1: now also IC$1.25, J4.1; no longer IC$1.2, J1.3
- net SRV2: now also IC$1.26, J4.2; no longer IC$1.25, J4.1
Routing:
- net 12V: track 33.1 -> 51.2 mm, vias 2 -> 0
- net SRV1: track 32.1 -> 17.0 mm
- net SRV3: track 14.8 -> 0.00 mm
- net 3_3V: track 66.2 -> 74.9 mm, vias 1 -> 15
- net LED: track 52.9 -> 47.9 mm
- net 5V: track 102.5 -> 105.5 mm, vias 0 -> 26
- net SRV2: track 17.0 -> 14.8 mm
- added copper zone on layer 16, net 3_3V
- added copper zone on layer 16, net 5V
Other:
- board text added: "1 2"
- board text added: "NC"
- board text removed: "1 2 3"
- board text removed: "LED"

Commit message: save
Other:
- board text removed: "NC"
Changed lines of the file:
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@@
 <grid distance="8" unitdist="mil" unit="mil" style="lines" multiple="1" display="yes" altdistance="4" altunitdist="mil" altunit="mil"/>
 <layers>
-<layer number="1" name="Top" color="4" fill="1" visible="yes" active="yes"/>
+<layer number="1" name="Top" color="4" fill="1" visible="no" active="yes"/>
 <layer number="16" name="Bottom" color="1" fill="1" visible="yes" active="yes"/>
 <layer number="17" name="Pads" color="2" fill="1" visible="yes" active="yes"/>
@@
 <layer number="19" name="Unrouted" color="6" fill="1" visible="yes" active="yes"/>
 <layer number="20" name="Dimension" color="24" fill="1" visible="yes" active="yes"/>
-<layer number="21" name="tPlace" color="7" fill="1" visible="yes" active="yes"/>
+<layer number="21" name="tPlace" color="7" fill="1" visible="no" active="yes"/>
 <layer number="22" name="bPlace" color="7" fill="1" visible="yes" active="yes"/>
-<layer number="23" name="tOrigins" color="15" fill="1" visible="yes" active="yes"/>
+<layer number="23" name="tOrigins" color="15" fill="1" visible="no" active="yes"/>
 <layer number="24" name="bOrigins" color="15" fill="1" visible="yes" active="yes"/>
-<layer number="25" name="tNames" color="7" fill="1" visible="yes" active="yes"/>
+<layer number="25" name="tNames" color="7" fill="1" visible="no" active="yes"/>
 <layer number="26" name="bNames" color="7" fill="1" visible="yes" active="yes"/>
-<layer number="27" name="tValues" color="7" fill="1" visible="yes" active="yes"/>
-<layer number="28" name="bValues" color="7" fill="1" visible="yes" active="yes"/>
+<layer number="27" name="tValues" color="7" fill="1" visible="no" active="yes"/>
+<layer number="28" name="bValues" color="7" fill="1" visible="no" active="yes"/>
 <layer number="29" name="tStop" color="7" fill="3" visible="no" active="yes"/>
 <layer number="30" name="bStop" color="7" fill="6" visible="no" active="yes"/>
@@
 <layer number="37" name="tTest" color="7" fill="1" visible="no" active="yes"/>
 <layer number="38" name="bTest" color="7" fill="1" visible="no" active="yes"/>
-<layer number="39" name="tKeepout" color="4" fill="11" visible="yes" active="yes"/>
+<layer number="39" name="tKeepout" color="4" fill="11" visible="no" active="yes"/>
 <layer number="40" name="bKeepout" color="1" fill="11" visible="yes" active="yes"/>
-<layer number="41" name="tRestrict" color="4" fill="10" visible="yes" active="yes"/>
+<layer number="41" name="tRestrict" color="4" fill="10" visible="no" active="yes"/>
 <layer number="42" name="bRestrict" color="1" fill="10" visible="yes" active="yes"/>
 <layer number="43" name="vRestrict" color="2" fill="10" visible="no" active="yes"/>
-<layer number="44" name="Drills" color="7" fill="1" visible="yes" active="yes"/>
+<layer number="44" name="Drills" color="7" fill="1" visible="no" active="yes"/>
 <layer number="45" name="Holes" color="7" fill="1" visible="yes" active="yes"/>
 <layer number="46" name="Milling" color="3" fill="1" visible="no" active="yes"/>
@@
 <layer number="49" name="Reference" color="7" fill="1" visible="no" active="yes"/>
 <layer number="50" name="dxf" color="7" fill="1" visible="no" active="no"/>
-<layer number="51" name="tDocu" color="7" fill="1" visible="yes" active="yes"/>
+<layer number="51" name="tDocu" color="7" fill="1" visible="no" active="yes"/>
 <layer number="52" name="bDocu" color="7" fill="1" visible="yes" active="yes"/>
 <layer number="53" name="tGND_GNDA" color="7" fill="9" visible="no" active="no"/>
@@
 <text x="19.9136" y="17.8816" size="1.27" layer="26" font="vector" ratio="11" rot="MR90">Revision:</text>
 <text x="19.9136" y="26.0096" size="1.2" layer="26" font="vector" rot="SMR90">&gt;CREVISION</text>
-<text x="47.3456" y="35.3568" size="1.016" layer="26" font="vector" rot="MR0">VCC</text>
-<text x="47.3456" y="37.9984" size="1.016" layer="26" font="vector" rot="MR0">GND</text>
-<text x="47.1424" y="40.64" size="1.016" layer="26" font="vector" rot="MR0">NC</text>
+<text x="47.1424" y="37.9984" size="1.016" layer="26" font="vector" rot="MR0">VCC</text>
+<text x="47.1424" y="40.64" size="1.016" layer="26" font="vector" rot="MR0">GND</text>
 <text x="47.1424" y="43.0784" size="0.8128" layer="26" font="vector" rot="MR0">CAN_L</text>
 <text x="47.1424" y="45.5168" size="0.8128" layer="26" font="vector" rot="MR0">CAN_H</text>
