File: data/Franks Flightsim Boards/Controler 2_25/Controler 2_25.sch (EAGLE design)
At the start: 16 parts, among them IC1 3_3V, IC2 5V, J3 External, J4 FEMALE 2x3

Commit message: backup
Parts:
- removed J1: (no value), SparkFun-Connectors:CONN_03
- J3: value External -> 22-27-2041-04; device con-molex:22-27-2051-05 -> con-molex:22-27-2041-04
Connections:
- removed net SRV3: IC$1.P13/R14, J4.2
- net 12V: now also J3-4.S; no longer J3-5.S
- net 3_3V: now also IC$2.VCC
- net 5V: no longer IC$2.VCC, J1.2
- net GND: now also J3-3.S; no longer J1.1, J3-4.S
- net LED: now also IC$1.P12; no longer J3-3.S
- net SRV1: now also IC$1.P15/R13, J4.1; no longer IC$1.P12, J1.3
- net SRV2: now also IC$1.P13/R14, J4.2; no longer IC$1.P15/R13, J4.1
Other:
- moved on the sheet: J3-1, J3-2, J3-3, J3-4
Changed lines of the file:
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@@
 <class number="4" name="5V" width="0.508" drill="0">
 </class>
-<class number="5" name="LED" width="0.508" drill="0">
+<class number="5" name="LED" width="0.254" drill="0">
 </class>
 </classes>
@@
 <part name="C3" library="resistor" library_urn="urn:adsk.eagle:library:348" deviceset="C-EU" device="C1206" package3d_urn="urn:adsk.eagle:package:26140/1" value="100nF"/>
 <part name="J2" library="SparkFun-Connectors" library_urn="urn:adsk.eagle:library:513" deviceset="CONN_16" device="" package3d_urn="urn:adsk.eagle:package:38258/1"/>
-<part name="J3" library="con-molex" library_urn="urn:adsk.eagle:library:165" deviceset="22-?-05" device="27-2051" value="External"/>
-<part name="J1" library="SparkFun-Connectors" library_urn="urn:adsk.eagle:library:513" deviceset="CONN_03" device="" package3d_urn="urn:adsk.eagle:package:38063/1"/>
 <part name="J4" library="SparkFun-Connectors" library_urn="urn:adsk.eagle:library:513" deviceset="CONN_03X2" device="FEMALE" package3d_urn="urn:adsk.eagle:package:38016/1" value="FEMALE 2x3"/>
 <part name="C5" library="resistor" library_urn="urn:adsk.eagle:library:348" deviceset="CPOL-EU" device="153CLV-0605" package3d_urn="urn:adsk.eagle:package:25889/1" value="47uF"/>
 <part name="C6" library="resistor" library_urn="urn:adsk.eagle:library:348" deviceset="C-EU" device="C1206" package3d_urn="urn:adsk.eagle:package:26140/1" value="100nF"/>
+<part name="J3" library="con-molex" library_urn="urn:adsk.eagle:library:165" deviceset="22-?-04" device="27-2041"/>
 </parts>
 <sheets>
@@
 <instance part="C3" gate="G$1" x="175.26" y="10.16"/>
 <instance part="J2" gate="G$1" x="98.552" y="87.63"/>
-<instance part="J3" gate="-1" x="109.22" y="-5.08" rot="R180"/>
-<instance part="J3" gate="-2" x="109.22" y="0" rot="R180"/>
-<instance part="J3" gate="-3" x="109.22" y="5.08" rot="R180"/>
-<instance part="J3" gate="-4" x="109.22" y="10.16" rot="R180"/>
-<instance part="J3" gate="-5" x="109.22" y="15.24" rot="R180"/>
-<instance part="J1" gate="J$1" x="0" y="38.1" rot="MR180"/>
 <instance part="J4" gate="G$1" x="0" y="55.88"/>
 <instance part="C5" gate="G$1" x="132.08" y="10.16"/>
 <instance part="C6" gate="G$1" x="218.44" y="10.16"/>
+<instance part="J3" gate="-1" x="106.68" y="7.62" smashed="yes" rot="MR0">
+<attribute name="NAME" x="104.14" y="6.858" size="1.524" layer="95" rot="MR0"/>
+<attribute name="VALUE" x="104.902" y="3.937" size="1.778" layer="96" rot="MR0"/>
+</instance>
+<instance part="J3" gate="-2" x="106.68" y="10.16" rot="MR0"/>
+<instance part="J3" gate="-3" x="106.68" y="12.7" rot="MR0"/>
+<instance part="J3" gate="-4" x="106.68" y="15.24" rot="MR0"/>
 </instances>
 <busses>
@@
 <wire x1="142.24" y1="10.16" x2="142.24" y2="15.24" width="0.1524" layer="91"/>
 <wire x1="142.24" y1="15.24" x2="147.32" y2="15.24" width="0.1524" layer="91"/>
-<wire x1="111.76" y1="15.24" x2="132.08" y2="15.24" width="0.1524" layer="91"/>
 <junction x="142.24" y="15.24"/>
 <wire x1="132.08" y1="15.24" x2="142.24" y2="15.24" width="0.1524" layer="91"/>
@@
 <wire x1="187.96" y1="15.24" x2="185.42" y2="15.24" width="0.1524" layer="91"/>
 <wire x1="185.42" y1="20.32" x2="185.42" y2="15.24" width="0.1524" layer="91"/>
-<pinref part="J3" gate="-5" pin="S"/>
 <pinref part="C5" gate="G$1" pin="+"/>
 <wire x1="132.08" y1="12.7" x2="132.08" y2="15.24" width="0.1524" layer="91"/>
+<pinref part="J3" gate="-4" pin="S"/>
+<wire x1="132.08" y1="15.24" x2="109.22" y2="15.24" width="0.1524" layer="91"/>
 <junction x="132.08" y="15.24"/>
 </segment>
@@
 <wire x1="165.1" y1="7.62" x2="165.1" y2="2.54" width="0.1524" layer="91"/>
 <junction x="165.1" y="2.54"/>
-<pinref part="J3" gate="-4" pin="S"/>
-<wire x1="111.76" y1="10.16" x2="124.46" y2="10.16" width="0.1524" layer="91"/>
-<wire x1="124.46" y1="10.16" x2="124.46" y2="2.54" width="0.1524" layer="91"/>
 <pinref part="C5" gate="G$1" pin="-"/>
 <wire x1="132.08" y1="5.08" x2="132.08" y2="2.54" width="0.1524" layer="91"/>
@@
 <wire x1="218.44" y1="2.54" x2="208.28" y2="2.54" width="0.1524" layer="91"/>
 <junction x="208.28" y="2.54"/>
+<wire x1="124.46" y1="2.54" x2="124.46" y2="12.7" width="0.1524" layer="91"/>
+<pinref part="J3" gate="-3" pin="S"/>
+<wire x1="124.46" y1="12.7" x2="109.22" y2="12.7" width="0.1524" layer="91"/>
 </segment>
 <segment>
@@
 <wire x1="10.16" y1="48.26" x2="15.24" y2="48.26" width="0.1524" layer="91"/>
 <junction x="10.16" y="48.26"/>
-<wire x1="10.16" y1="48.26" x2="10.16" y2="40.64" width="0.1524" layer="91"/>
-<pinref part="J1" gate="J$1" pin="1"/>
-<wire x1="10.16" y1="40.64" x2="7.62" y2="40.64" width="0.1524" layer="91"/>
 </segment>
 </net>
@@
 </segment>
 <segment>
-<pinref part="IC$2" gate="G$1" pin="VCC"/>
-<wire x1="60.96" y1="-20.32" x2="58.42" y2="-20.32" width="0.1524" layer="91"/>
-<label x="58.42" y="-20.32" size="1.27" layer="95" ratio="7" rot="MR0" xref="yes"/>
-</segment>
-<segment>
 <pinref part="J2" gate="G$1" pin="15"/>
 <wire x1="108.712" y1="102.87" x2="111.76" y2="102.87" width="0.1524" layer="91"/>
@@
 <junction x="12.7" y="45.72"/>
 <label x="15.24" y="45.72" size="1.27" layer="95" xref="yes"/>
-<wire x1="12.7" y1="45.72" x2="12.7" y2="38.1" width="0.1524" layer="91"/>
-<pinref part="J1" gate="J$1" pin="2"/>
-<wire x1="12.7" y1="38.1" x2="7.62" y2="38.1" width="0.1524" layer="91"/>
 </segment>
 </net>
@@
 <label x="111.76" y="105.41" size="1.27" layer="95" ratio="7" xref="yes"/>
 </segment>
+<segment>
+<pinref part="IC$2" gate="G$1" pin="VCC"/>
+<wire x1="60.96" y1="-20.32" x2="58.42" y2="-20.32" width="0.1524" layer="91"/>
+<label x="58.42" y="-20.32" size="1.27" layer="95" rot="R180" xref="yes"/>
+</segment>
 </net>
 <net name="LED" class="5">
-<segment>
-<pinref part="J3" gate="-3" pin="S"/>
-<wire x1="111.76" y1="5.08" x2="114.3" y2="5.08" width="0.1524" layer="91"/>
-<label x="114.3" y="5.08" size="1.778" layer="95" xref="yes"/>
-</segment>
 <segment>
 <pinref part="J2" gate="G$1" pin="14"/>
@@
 <label x="111.76" y="100.33" size="1.27" layer="95" ratio="7" xref="yes"/>
 </segment>
+<segment>
+<pinref part="IC$1" gate="G$1" pin="P12"/>
+<wire x1="73.66" y1="104.14" x2="78.74" y2="104.14" width="0.1524" layer="91"/>
+<label x="78.74" y="104.14" size="1.27" layer="95" xref="yes"/>
+</segment>
 </net>
 <net name="P35" class="0">
@@
 </segment>
 </net>
-<net name="SRV3" class="0">
+<net name="SRV2" class="0">
 <segment>
 <pinref part="IC$1" gate="G$1" pin="P13/R14"/>
@@
 </segment>
 </net>
-<net name="SRV2" class="0">
-<segment>
-<pinref part="IC$1" gate="G$1" pin="P15/R13"/>
-<wire x1="38.1" y1="104.14" x2="33.02" y2="104.14" width="0.1524" layer="91"/>
-<label x="33.02" y="104.14" size="1.27" layer="95" ratio="7" rot="R180" xref="yes"/>
-</segment>
-<segment>
-<label x="-10.16" y="58.42" size="1.27" layer="95" rot="MR0" xref="yes"/>
-<pinref part="J4" gate="G$1" pin="1"/>
-<wire x1="-10.16" y1="58.42" x2="-7.62" y2="58.42" width="0.1524" layer="91"/>
-</segment>
-</net>
-<net name="SRV1" class="0">
-<segment>
-<pinref part="IC$1" gate="G$1" pin="P12"/>
-<wire x1="73.66" y1="104.14" x2="78.74" y2="104.14" width="0.1524" layer="91"/>
-<label x="78.74" y="104.14" size="1.27" layer="95" ratio="7" rot="MR180" xref="yes"/>
-</segment>
-<segment>
-<label x="10.16" y="35.56" size="1.27" layer="95" xref="yes"/>
-<pinref part="J1" gate="J$1" pin="3"/>
-<wire x1="10.16" y1="35.56" x2="7.62" y2="35.56" width="0.1524" layer="91"/>
-</segment>
-</net>
 <net name="P14" class="0">
 <segment>
@@
 <net name="N$2" class="0">
 <segment>
-<pinref part="J3" gate="-1" pin="S"/>
 <pinref part="R2" gate="G$1" pin="2"/>
 <wire x1="99.06" y1="-10.16" x2="99.06" y2="-12.7" width="0.1524" layer="91"/>
@@
 <wire x1="99.06" y1="-10.16" x2="116.84" y2="-10.16" width="0.1524" layer="91"/>
 <junction x="99.06" y="-10.16"/>
-<wire x1="116.84" y1="-10.16" x2="116.84" y2="-5.08" width="0.1524" layer="91"/>
-<wire x1="111.76" y1="-5.08" x2="114.3" y2="-5.08" width="0.1524" layer="91"/>
-<wire x1="114.3" y1="-5.08" x2="116.84" y2="-5.08" width="0.1524" layer="91"/>
+<wire x1="116.84" y1="-10.16" x2="116.84" y2="7.62" width="0.1524" layer="91"/>
+<pinref part="J3" gate="-1" pin="S"/>
+<wire x1="116.84" y1="7.62" x2="109.22" y2="7.62" width="0.1524" layer="91"/>
 </segment>
 </net>
 <net name="N$3" class="0">
 <segment>
-<pinref part="J3" gate="-2" pin="S"/>
 <pinref part="R2" gate="G$1" pin="1"/>
 <wire x1="99.06" y1="-25.4" x2="99.06" y2="-22.86" width="0.1524" layer="91"/>
@@
 <wire x1="93.98" y1="-20.32" x2="93.98" y2="-25.4" width="0.1524" layer="91"/>
 <wire x1="93.98" y1="-25.4" x2="99.06" y2="-25.4" width="0.1524" layer="91"/>
-<wire x1="119.38" y1="-25.4" x2="119.38" y2="0" width="0.1524" layer="91"/>
+<wire x1="119.38" y1="-25.4" x2="119.38" y2="10.16" width="0.1524" layer="91"/>
 <wire x1="99.06" y1="-25.4" x2="119.38" y2="-25.4" width="0.1524" layer="91"/>
 <junction x="99.06" y="-25.4"/>
-<wire x1="111.76" y1="0" x2="119.38" y2="0" width="0.1524" layer="91"/>
-</segment>
-</net>
+<pinref part="J3" gate="-2" pin="S"/>
+<wire x1="119.38" y1="10.16" x2="109.22" y2="10.16" width="0.1524" layer="91"/>
+</segment>
+</net>
+<net name="SRV1" class="0">
+<segment>
+<label x="-10.16" y="58.42" size="1.27" layer="95" rot="MR0" xref="yes"/>
+<pinref part="J4" gate="G$1" pin="1"/>
+<wire x1="-10.16" y1="58.42" x2="-7.62" y2="58.42" width="0.1524" layer="91"/>
+</segment>
+<segment>
+<pinref part="IC$1" gate="G$1" pin="P15/R13"/>
+<wire x1="38.1" y1="104.14" x2="33.02" y2="104.14" width="0.1524" layer="91"/>
+<label x="33.02" y="104.14" size="1.27" layer="95" ratio="7" rot="R180" xref="yes"/>
+</segment>
+</net>
