File: data/Franks Flightsim Boards/Motor Board 2_25/Motor_board_2_5.sch (EAGLE design)
At the start: 9 parts, among them IC1 VID66-08, J4 LEDS

Commit message: Update dev status
Parts:
- removed J4: LEDS, con-molex:22-27-2021-02
- added D1, D2: (no value), SparkFun-LED:LED-3MM-NO_SILK
- added R1: 220, resistor:R-EU_0204/7
- C1: device SparkFun-Capacitors:22UF-POLAR-PANASONIC_C-35V-20% -> rcl:CPOL-EU153CLV-0605
- C3, C4: device rcl:C-EUC0805 -> rcl:C-EUC1206K
- R9: device resistor:R-EU_M1206 -> resistor:R-EU_M0805
- STEPPER1, STEPPER2: value VID29 -> VID29BKA30-R5; device Franks:VID29 -> Franks:VID29BKA30-R5
Connections:
- net OUT1B renamed OUT_3B
- net OUT2B renamed OUT_4B
- net OUT3B renamed OUT_1B
- net OUT4B renamed OUT_2B
- removed net OUT1A: IC1.OUT3A, STEPPER1.M1A
- removed net OUT2A: IC1.OUT4A, STEPPER1.M2A
- removed net OUT3A: IC1.OUT1A, STEPPER1.M3A
- removed net OUT4A: IC1.OUT2A, STEPPER1.M4A
- new net N$1: D1.A, D2.A, R1.2
- new net OUT_1A: IC1.OUT1A, STEPPER1.M4A
- new net OUT_2A: IC1.OUT2A, STEPPER1.M3A
- new net OUT_3A: IC1.OUT3A, STEPPER1.M2A
- new net OUT_4A: IC1.OUT4A, STEPPER1.M1A
- net GND: now also D1.C, D2.C; no longer J4-2.S
- net LED: now also R1.1; no longer J4-1.S
Other:
- moved on the sheet: C1, C3, C4, R9
