File: data/Franks Flightsim Boards/Motor Board 2_25/Motor_board_2_5.brd (EAGLE design)
At the start: 60 x 60 mm, 14 parts, among them IC1 VID66-08, J4 LEDS

Commit message: Update dev status
Parts:
- removed J4: LEDS, con-molex:6410-02
- added D1, D2: (no value), SparkFun-LED:LED_3MM-NS
- added R1: 220, resistor:0204/7
- C1: device SparkFun-Capacitors:PANASONIC_C -> rcl:153CLV-0605
- C3, C4: device rcl:C0805 -> rcl:C1206K
- R9: device resistor:M1206 -> resistor:M0805
- STEPPER1, STEPPER2: value VID29 -> VID29BKA30-R5; device Franks:VID29_STEPPER_BACK -> Franks:BKA30-R5
- moved U$9 19.4 mm to (30.1, 18.6)
- moved C3 16.7 mm to (34.1, 52.7), turned to 0 degrees
- moved C1 9.55 mm to (21.9, 50.4), flipped to the bottom, turned to 90 degrees
- moved R9 0.81 mm to (37.2, 46.9)
- moved C4 0.73 mm to (30.9, 34.6)
Connections:
- net OUT1B renamed OUT_3B
- net OUT2B renamed OUT_4B
- net OUT3B renamed OUT_1B
- net OUT4B renamed OUT_2B
- removed net OUT1A: IC1.6, STEPPER1.M1A
- removed net OUT2A: IC1.5, STEPPER1.M2A
- removed net OUT3A: IC1.3, STEPPER1.M3A
- removed net OUT4A: IC1.4, STEPPER1.M4A
- new net N$1: D1.A, D2.A, R1.2
- new net OUT_1A: IC1.3, STEPPER1.M4A
- new net OUT_2A: IC1.4, STEPPER1.M3A
- new net OUT_3A: IC1.6, STEPPER1.M2A
- new net OUT_4A: IC1.5, STEPPER1.M1A
- net GND: now also D1.K, D2.K; no longer J4.2
- net LED: now also R1.1; no longer J4.1
Routing:
- net LED: track 11.4 -> 54.4 mm, vias 0 -> 1
- net OUT_3A: track 0.00 -> 32.3 mm, vias 0 -> 2
- net OUT2A: track 31.6 -> 0.00 mm
- net N$1: track 0.00 -> 30.2 mm
- net OUT_4A: track 0.00 -> 29.0 mm
- net OUT1A: track 27.5 -> 0.00 mm
- net OUT_2A: track 0.00 -> 18.2 mm
- net OUT3A: track 18.1 -> 0.00 mm
- net OUT_1A: track 0.00 -> 11.6 mm, vias 0 -> 2
- net OUT4A: track 9.57 -> 0.00 mm
- net 5V: track 51.5 -> 53.3 mm, vias 3 -> 2

Commit message: update and backup
Update
Parts:
- moved U$9 0.20 mm to (30.1, 18.4), turned to 177.2 degrees
Changed lines of the file:
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@@
 <wire x1="60" y1="60" x2="0" y2="60" width="0" layer="20"/>
 <wire x1="0" y1="60" x2="0" y2="0" width="0" layer="20"/>
-<text x="19.2144" y="14.8928" size="1.4224" layer="25" font="vector" ratio="11" rot="R180" align="bottom-right">&gt;CProject</text>
-<text x="26.808" y="11.096" size="1.27" layer="25" font="vector" ratio="11" rot="R180" align="bottom-right">&gt;CREVISION</text>
-<text x="19.2144" y="12.8928" size="1.27" layer="25" font="vector" ratio="11" rot="R180" align="bottom-right">&gt;DRAWING_NAME</text>
-<text x="19.2144" y="11.096" size="1.27" layer="25" font="vector" ratio="11" rot="R180" align="bottom-right">Revision:</text>
+<text x="40.9568" y="8.7968" size="1.4224" layer="25" font="vector" ratio="11" rot="SR180" align="top-left">&gt;CProject</text>
+<text x="33.3104" y="12.7216" size="1.27" layer="25" font="vector" ratio="11" rot="SR180" align="top-left">&gt;CREVISION</text>
+<text x="40.9568" y="10.8608" size="1.27" layer="25" font="vector" ratio="11" rot="SR180" align="top-left">&gt;DRAWING_NAME</text>
+<text x="40.9568" y="12.7216" size="1.27" layer="25" font="vector" ratio="11" rot="SR180" align="top-left">Revision:</text>
 </plain>
 <attributes>
 <attribute name="CPROJECT" value="Franks Flightsim Boards"/>
-<attribute name="CREVISION" value="v0.2"/>
+<attribute name="CREVISION" value="v0.3"/>
 </attributes>
 <variantdefs>
@@
 <elements>
 <element name="STEPPER1" library="Franks" package="BKA30-R5" value="VID29BKA30-R5" x="9" y="30" smashed="yes" rot="MR90">
-<attribute name="NAME" x="20.35" y="21.65" size="1.27" layer="22" rot="MR90"/>
+<attribute name="NAME" x="7.9548" y="34.858" size="1.27" layer="22" rot="SMR180"/>
 </element>
 <element name="STEPPER2" library="Franks" package="BKA30-R5" value="VID29BKA30-R5" x="51" y="30" smashed="yes" rot="MR270">
-<attribute name="NAME" x="39.65" y="38.35" size="1.27" layer="22" rot="MR270"/>
+<attribute name="NAME" x="42.9012" y="34.4892" size="1.27" layer="22" rot="SMR180"/>
 </element>
 <element name="U$1" library="mechanics_v5" package="M2.0_SW4.0_HOLE" value="" x="3.5" y="45" locked="yes"/>
@@
 <element name="R9" library="resistor" library_urn="urn:adsk.eagle:library:348" package="M0805" package3d_urn="urn:adsk.eagle:package:26079/1" value="1k" x="37.2364" y="46.9392" rot="R90"/>
 <element name="C1" library="rcl" library_urn="urn:adsk.eagle:library:334" package="153CLV-0605" package3d_urn="urn:adsk.eagle:package:23398/1" value="22uF" x="21.9456" y="50.3936" smashed="yes" rot="MR90">
-<attribute name="NAME" x="19.3294" y="54.4576" size="1.016" layer="26" font="vector" ratio="11" rot="MR0" align="bottom-center"/>
+<attribute name="NAME" x="25.019" y="55.0672" size="1.016" layer="26" font="vector" ratio="11" rot="SMR180" align="bottom-center"/>
 <attribute name="SPICEPREFIX" value="C" x="21.9456" y="50.3936" size="1.778" layer="28" rot="MR90" display="off"/>
 </element>
 <element name="C3" library="rcl" library_urn="urn:adsk.eagle:library:334" package="C1206K" package3d_urn="urn:adsk.eagle:package:23682/2" value="100nF" x="34.1376" y="52.7304" smashed="yes">
-<attribute name="NAME" x="34.29" y="54.2036" size="1.27" layer="25" font="vector"/>
+<attribute name="NAME" x="38.354" y="53.3908" size="1.27" layer="25" font="vector" rot="SR180"/>
 <attribute name="SPICEPREFIX" value="C" x="29.0576" y="45.1104" size="1.778" layer="27" display="off"/>
-<attribute name="VALUE" x="36.7284" y="52.0192" size="1.27" layer="27"/>
-</element>
-<element name="C4" library="rcl" library_urn="urn:adsk.eagle:library:334" package="C1206K" package3d_urn="urn:adsk.eagle:package:23682/2" value="100nF" x="30.9372" y="34.6456">
+<attribute name="VALUE" x="38.9636" y="51.4096" size="1.27" layer="27" rot="SR180"/>
+</element>
+<element name="C4" library="rcl" library_urn="urn:adsk.eagle:library:334" package="C1206K" package3d_urn="urn:adsk.eagle:package:23682/2" value="100nF" x="30.9372" y="34.6456" smashed="yes">
+<attribute name="NAME" x="35.0268" y="34.7296" size="1.016" layer="25" rot="SR180"/>
 <attribute name="SPICEPREFIX" value="C" x="30.9372" y="34.6456" size="1.778" layer="27" display="off"/>
-</element>
-<element name="U$9" library="SparkFun-Aesthetics" library_urn="urn:adsk.eagle:library:507" package="OSHW-LOGO-L" package3d_urn="urn:adsk.eagle:package:37097/1" value="" x="30.1392" y="18.5564" smashed="yes" rot="R357.2"/>
+<attribute name="VALUE" x="33.8076" y="33.1552" size="1.016" layer="27" rot="SR180"/>
+</element>
+<element name="U$9" library="SparkFun-Aesthetics" library_urn="urn:adsk.eagle:library:507" package="OSHW-LOGO-L" package3d_urn="urn:adsk.eagle:package:37097/1" value="" x="30.1392" y="18.3532" smashed="yes" rot="R177.2"/>
 <element name="D1" library="SparkFun-LED" library_urn="urn:adsk.eagle:library:529" package="LED_3MM-NS" package3d_urn="urn:adsk.eagle:package:39356/1" value="" x="15.75" y="5.328" smashed="yes" rot="R150">
-<attribute name="NAME" x="14.4038" y="2.941865625" size="1.016" layer="25" font="vector" ratio="11" rot="R150" align="bottom-center"/>
+<attribute name="NAME" x="15.8262" y="8.834665625" size="1.016" layer="25" font="vector" ratio="11" rot="SR180" align="bottom-center"/>
 <attribute name="VALUE" x="16.893" y="7.30773125" size="0.6096" layer="27" font="vector" ratio="20" rot="R150" align="top-center"/>
 </element>
 <element name="D2" library="SparkFun-LED" library_urn="urn:adsk.eagle:library:529" package="LED_3MM-NS" package3d_urn="urn:adsk.eagle:package:39356/1" value="" x="45.75" y="5.328" smashed="yes" rot="R30">
-<attribute name="NAME" x="44.4038" y="7.51093125" size="1.016" layer="25" font="vector" ratio="11" rot="R30" align="bottom-center"/>
+<attribute name="NAME" x="45.623" y="8.73013125" size="1.016" layer="25" font="vector" ratio="11" rot="SR183.9" align="bottom-center"/>
 <attribute name="VALUE" x="46.893" y="3.348265625" size="0.6096" layer="27" font="vector" ratio="20" rot="R30" align="top-center"/>
 </element>

Commit message: backup
Parts:
- moved D1 2.70 mm to (13.1, 5.86), turned to 145 degrees
- moved D2 1.27 mm to (46.9, 5.86), turned to 35 degrees
Routing:
- net N$1: track 30.2 -> 34.1 mm
Changed lines of the file:
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@@
 <setting verticaltext="up"/>
 </settings>
-<grid distance="8" unitdist="mil" unit="mil" style="lines" multiple="1" display="yes" altdistance="4" altunitdist="mil" altunit="mil"/>
+<grid distance="8" unitdist="mil" unit="mm" style="lines" multiple="1" display="yes" altdistance="4" altunitdist="mil" altunit="mm"/>
 <layers>
 <layer number="1" name="Top" color="4" fill="1" visible="yes" active="yes"/>
@@
 </element>
 <element name="U$9" library="SparkFun-Aesthetics" library_urn="urn:adsk.eagle:library:507" package="OSHW-LOGO-L" package3d_urn="urn:adsk.eagle:package:37097/1" value="" x="30.1392" y="18.3532" smashed="yes" rot="R177.2"/>
-<element name="D1" library="SparkFun-LED" library_urn="urn:adsk.eagle:library:529" package="LED_3MM-NS" package3d_urn="urn:adsk.eagle:package:39356/1" value="" x="15.75" y="5.328" smashed="yes" rot="R150">
-<attribute name="NAME" x="15.8262" y="8.834665625" size="1.016" layer="25" font="vector" ratio="11" rot="SR180" align="bottom-center"/>
-<attribute name="VALUE" x="16.893" y="7.30773125" size="0.6096" layer="27" font="vector" ratio="20" rot="R150" align="top-center"/>
-</element>
-<element name="D2" library="SparkFun-LED" library_urn="urn:adsk.eagle:library:529" package="LED_3MM-NS" package3d_urn="urn:adsk.eagle:package:39356/1" value="" x="45.75" y="5.328" smashed="yes" rot="R30">
-<attribute name="NAME" x="45.623" y="8.73013125" size="1.016" layer="25" font="vector" ratio="11" rot="SR183.9" align="bottom-center"/>
-<attribute name="VALUE" x="46.893" y="3.348265625" size="0.6096" layer="27" font="vector" ratio="20" rot="R30" align="top-center"/>
+<element name="D1" library="SparkFun-LED" library_urn="urn:adsk.eagle:library:529" package="LED_3MM-NS" package3d_urn="urn:adsk.eagle:package:39356/1" value="" x="13.1" y="5.86" smashed="yes" rot="R145">
+<attribute name="NAME" x="13.481534375" y="9.346678125" size="1.016" layer="25" font="vector" ratio="11" rot="SR175" align="bottom-center"/>
+<attribute name="VALUE" x="14.41119375" y="7.732578125" size="0.6096" layer="27" font="vector" ratio="20" rot="R145" align="top-center"/>
+</element>
+<element name="D2" library="SparkFun-LED" library_urn="urn:adsk.eagle:library:529" package="LED_3MM-NS" package3d_urn="urn:adsk.eagle:package:39356/1" value="" x="46.9" y="5.86" smashed="yes" rot="R35">
+<attribute name="NAME" x="46.476965625" y="9.2381125" size="1.016" layer="25" font="vector" ratio="11" rot="SR188.9" align="bottom-center"/>
+<attribute name="VALUE" x="48.21119375" y="3.987415625" size="0.6096" layer="27" font="vector" ratio="20" rot="R35" align="top-center"/>
 </element>
 <element name="R1" library="resistor" library_urn="urn:adsk.eagle:library:348" package="0204/7" package3d_urn="urn:adsk.eagle:package:25945/1" value="220" x="29.2608" y="7.5184" smashed="yes">
@@
 <contactref element="D1" pad="A"/>
 <contactref element="D2" pad="A"/>
-<wire x1="33.0708" y1="7.5184" x2="35.8962" y2="4.693" width="0.8128" layer="16"/>
-<wire x1="35.8962" y1="4.693" x2="44.650146875" y2="4.693" width="0.8128" layer="16"/>
-<wire x1="33.0708" y1="7.5184" x2="30.4486" y2="4.693" width="0.8128" layer="16"/>
-<wire x1="30.4486" y1="4.693" x2="16.84985" y2="4.693" width="0.8128" layer="16"/>
+<wire x1="33.0708" y1="7.5184" x2="34.8802" y2="5.0994" width="0.8128" layer="16"/>
+<wire x1="34.8802" y1="5.0994" x2="45.859675" y2="5.13155625" width="0.8128" layer="16"/>
+<wire x1="33.0708" y1="7.5184" x2="31.2614" y2="5.0994" width="0.8128" layer="16"/>
+<wire x1="31.2614" y1="5.0994" x2="14.140321875" y2="5.13155625" width="0.8128" layer="16"/>
 </signal>
 <signal name="OUT_2A">
