File: data/Franks Flightsim Boards/Controler 2_25-ESP32/Controler 2_25.brd (EAGLE design)
At the start: 60 x 60 mm, 20 parts, among them IC1 3_3V, IC2 5V, J3 External, J4 FEMALE 2x3

Commit message: daily sync
Parts:
- removed IC$1: LOLIN32LITE, Franks:LOLIN32LITE
- added F1: 0.75A 16V, fuses:1812L
- added IC3: ESP-WROOM32, Franks:ESP-WROOM32
- added J5: 22-27-2031-03, con-molex:6410-03
- added LED1: LG_T679-E1F1-1, led:PLCC2
- added R3: 10k, resistor:M1206
- added R4: 220, resistor:M1206
- added S1: RESET, SparkFun-Switches:TACTILE_SWITCH_SMD_4.6X2.8MM
- added S2: FLASH, SparkFun-Switches:TACTILE_SWITCH_SMD_4.6X2.8MM
- J2: value (none) -> BUS
- J3: value External -> 22-27-2041-04; device con-molex:6410-05 -> con-molex:6410-04
- moved U$10 28.9 mm to (50.5, 5.92)
- moved J4 12.0 mm to (27.2, 9.09)
- moved IC1 1.63 mm to (39.2, 26.0)
- moved C2 1.42 mm to (51.4, 24.4)
- moved C3 1.22 mm to (46.9, 24.6)
- moved C1 1.18 mm to (51.2, 31.3)
- moved J3 1.02 mm to (50.8, 42.1)
Connections:
- removed net CAN_D: IC$1.20, IC$2.1
- removed net P36: IC$1.13
- removed net P39: IC$1.12
- removed net SRV1: IC$1.25, J4.1
- removed net SRV2: IC$1.26, J4.2
- new net CAN_T: IC$2.1, IC3.28
- new net N$4: LED1.A, R4.1
- new net N$5: F1.1, J3.4
- new net N$6: IC3.5
- new net N$7: IC3.4
- new net P06: IC3.20, J2.3
- new net P07: IC3.21, J2.2
- new net P08: IC3.22
- new net P09: IC3.17, J2.6
- new net P10: IC3.18, J2.5
- new net P11: IC3.19, J2.4
- new net P13: IC3.16, R4.2
- new net P15: IC3.23, J4.2
- new net P21: IC3.33
- new net RESET: IC3.3, R3.1, S1.3, S1.4
- new net USB_RX: IC3.34, J5.2
- new net USB_TX: IC3.35, J5.1
- net 12V: now also F1.2; no longer J3.5
- net 3_3V: now also IC3.2, R3.2; no longer IC$1.14
- net CAN_R: now also IC3.27; no longer IC$1.21
- net GND: now also IC3.1, IC3.15, IC3.38, IC3.TP, J3.3, J5.3, LED1.C, S1.1, S1.2, S2.1, S2.2; no longer IC$1.1, J3.4
- net LED: now also IC3.14; no longer IC$1.2
- net P00: now also IC3.25, S2.3, S2.4; no longer IC$1.23, J2.3
- net P02: now also IC3.24, J4.1; no longer IC$1.24, J2.2
- net P04: now also IC3.26; no longer IC$1.22, J2.4
- net P05: now also IC3.29; no longer IC$1.19, J2.5
- net P14: now also IC3.13; no longer IC$1.3
- net P18: now also IC3.30; no longer IC$1.18, J2.6
- net P19: now also IC3.31; no longer IC$1.16, J2.8
- net P22: now also IC3.36; no longer IC$1.15
- net P23: now also IC3.37; no longer IC$1.17, J2.7
- net P25: now also IC3.10; no longer IC$1.6
- net P26: now also IC3.11, J2.8; no longer IC$1.5
- net P27: now also IC3.12, J2.7; no longer IC$1.4
- net P32: now also IC3.8; no longer IC$1.8
- net P33: now also IC3.9; no longer IC$1.7
- net P34: now also IC3.6; no longer IC$1.10
- net P35: now also IC3.7; no longer IC$1.9
Routing:
- net P07: track 0.00 -> 44.9 mm
- net P06: track 0.00 -> 41.2 mm
- net P09: track 0.00 -> 39.5 mm
- net P11: track 0.00 -> 38.8 mm
- net P10: track 0.00 -> 38.4 mm
- net P04: track 38.2 -> 0.00 mm
- net P19: track 37.5 -> 0.00 mm
- net P23: track 34.7 -> 0.00 mm
- net P27: track 0.00 -> 34.4 mm
- net P05: track 34.2 -> 0.00 mm
- net P13: track 0.00 -> 33.9 mm
- net P18: track 33.5 -> 0.00 mm
- net CAN_T: track 0.00 -> 31.9 mm, vias 0 -> 1
- net P26: track 0.00 -> 31.7 mm
- net P02: track 47.2 -> 15.8 mm
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Other:
- board text added: ">crevision"
- board text added: "Flash"
- board text added: "Reset"
- board text added: "Rx"
- board text added: "Tx"
- board text added: "USB"
- board text removed: ">CREVISION"
- board text removed: "NC"
