File: data/Franks Flightsim Boards/Controler 2_25-ESP32/Controler 2_25.sch (EAGLE design)
At the start: 13 parts, among them IC1 LD117AV33, IC2 LD117AV50, IC3 SN65HVD230, IC4 LOLIN32LITE, J1 EXTERN, J4 STEP_C

Commit message: daily sync
Parts:
- removed IC4: LOLIN32LITE, Franks:LOLIN32LITE
- removed J1: EXTERN, SparkFun-Connectors:CONN_05JST-VERT
- added C5: 47uF, resistor:CPOL-EU153CLV-0605
- added C6: 100nF, resistor:C-EUC1206
- added F1: 0.75A 16V, fuses:1812L
- added IC$2: SN65HVD230, Franks:SN65HVD230
- added J3: 22-27-2041-04, con-molex:22-27-2041-04
- added J5: 22-27-2031-03, con-molex:22-27-2031-03
- added LED1: LG_T679-E1F1-1, led:LG_T679-E1F1-1
- added R3: 10k, resistor:R-EU_M1206
- added R4: 220, resistor:R-EU_M1206
- added S1: RESET, SparkFun-Switches:MOMENTARY-SWITCH-SPST-2-SMD-4.6X2.8MM
- added S2: FLASH, SparkFun-Switches:MOMENTARY-SWITCH-SPST-2-SMD-4.6X2.8MM
- C1, C3: value 10uF -> 100nF; device resistor:CPOL-EU153CLV-0605 -> resistor:C-EUC1206
- C2, C4: value 100nF -> 47uF; device resistor:C-EUC0805 -> resistor:CPOL-EUCT3528
- IC1: value LD117AV33 -> 3_3V; device v-reg:LD117AV33 -> SparkFun-IC-Power:V_REG_LM1117SOT223
- IC2: value LD117AV50 -> 5V; device v-reg:LD117AV50 -> SparkFun-IC-Power:V_REG_LM1117SOT223
- IC3: value SN65HVD230 -> ESP-WROOM32; device Franks:SN65HVD230 -> Franks:ESP-WROOM32
- J2: value (none) -> BUS; device SparkFun-Connectors:CONN_20 -> SparkFun-Connectors:CONN_16
- J4: value STEP_C -> FEMALE 2x3; device SparkFun-Connectors:CONN_04JST-PTH-VERT -> SparkFun-Connectors:CONN_03X2FEMALE
- R1: value 120 -> 10k; device resistor:R-EU_0207/2V -> resistor:R-EU_M1206
- R2: value 10k -> 120; device resistor:R-EU_M1206 -> resistor:R-EU_R1210
Connections:
- removed net CAN_D: IC3.D, IC4.P17
- removed net N$49: IC3.CANL, J1.2, R1.1
- removed net P12: IC4.P12
- removed net P36: IC4.VP, J4.1
- removed net P39: IC4.VN, J4.2
- new net CAN_T: IC$2.D, IC3.TXD2/IO17
- new net N$2: IC$2.CANH, J3-1.S, R2.2
- new net N$3: IC$2.CANL, J3-2.S, R2.1
- new net N$5: F1.1, J3-4.S
- new net N$6: IC3.SVN/I039/A1C3
- new net N$7: IC3.SVP/I036/A1C0
- new net P06: IC3.SCK/IO6, J2.3
- new net P07: IC3.SDO/IO7, J2.2
- new net P08: IC3.SDI/IO8
- new net P09: IC3.SHD/IO9, J2.6
- new net P10: IC3.SWP/IO10, J2.5
- new net P11: IC3.SCS/IO11, J2.4
- new net P21: IC3.VSHD/IO21
- new net RESET: IC3.EN, R3.1, S1.3, S1.4
- new net USB_RX: IC3.RXD0/IO3, J5-2.S
- new net USB_TX: IC3.TXD0/IO1, J5-1.S
- net 12V: now also C1.1, C5.+, F1.2; no longer C2.1, C4.1, J1.5
- net 3_3V: now also C2.+, C3.1, IC$2.VCC, IC1.OUT@1, IC3.VCC, J2.16, R3.2; no longer C1.+, IC4.VCC, J2.20
- net 5V: now also C4.+, C6.1, IC2.OUT@1, J2.15, J4.3, J4.4; no longer C3.+, IC3.VCC, J2.19
- net CAN_R: now also IC$2.R, IC3.RXD2/IO16; no longer IC3.R, IC4.P16
- net GND: now also C1.2, C2.-, C3.2, C4.-, C5.-, C6.2, IC$2.GND, J3-3.S, J4.5, J4.6, J5-3.S, LED1.C, R1.1, S1.1, S1.2, S2.1, S2.2; no longer C1.-, C2.2, C3.-, C4.2, IC4.GND, J1.4, R2.1
- net LED: now also IC3.HSDO/A2C5/IO12, J2.14; no longer J1.3, J2.18
- net N$1: now also IC$2.RS, R1.2; no longer IC3.RS, R2.2
- net N$4: now also LED1.A, R4.1; no longer IC3.CANH, J1.1, R1.2
- net P00: now also IC3.BL/A2C1/IO0, S2.3, S2.4; no longer IC4.P0/R11, J2.7
- net P02: now also IC3.HSWP/A2C2/IO2, J4.1; no longer IC4.P2/R12, J2.9
- net P04: now also IC3.HSHD/A2C0/IO4; no longer IC4.P4/R10, J2.2
- net P05: now also IC3.VSCS/IO5; no longer IC4.P5, J2.3
- net P13: now also IC3.HSDI/A2C4/IO13, R4.2; no longer IC4.P13/R14, J4.4
- net P14: now also IC3.HSCK/A2C6/IO14; no longer IC4.P14, J2.10
- net P15: now also IC3.HSCS/A2C3/IO15, J4.2; no longer IC4.P15/R13, J4.3
- net P18: now also IC3.VSCK/IO18; no longer IC4.P18, J2.4
- net P19: now also IC3.VSDO/IO19; no longer IC4.P19, J2.6
- net P22: now also IC3.VSWP/IO22; no longer IC4.P22, J2.8
- net P23: now also IC3.VSDI/IO23; no longer IC4.P23, J2.5
- net P25: now also IC3.DAC1/A2C8/IO25, J2.9; no longer IC4.P25/R6/DAC1, J2.13
- net P26: now also IC3.DAC2/A2C9/IO26, J2.8; no longer IC4.P26/R2/DAC1, J2.12
- net P27: now also IC3.A2C7/IO27, J2.7; no longer IC4.P27, J2.11
- net P32: now also IC3.XIN32K/A1C4/IO32, J2.11; no longer IC4.P32, J2.15
- net P33: now also IC3.XOUT32K/A1C5/IO33, J2.10; no longer IC4.P33, J2.14
- net P34: now also IC3.A1C6/IO34, J2.13; no longer IC4.P34, J2.17
- net P35: now also IC3.A1C7/IO35, J2.12; no longer IC4.P35, J2.16
Other:
- moved on the sheet: R1, R2
