File: data/Franks Flightsim Boards/Controler 3_5/Controler 3_5.brd (EAGLE design)
At the start: 80 x 65 mm, 24 parts, among them IC1 SN65HVD230, IC2 LOLIN32LITE, IC3 LD117AV33, IC4 7805T, J1 External, J2 FEMALE 2x3, X1 BUS

Commit message: Update dev status
Parts:
- moved J3 5.58 mm to (35.0, 10.6), turned to 270 degrees
- moved C3 2.72 mm to (71.1, 8.13)
- moved D1 2.57 mm to (47.3, 17.8)
- moved IC3 2.44 mm to (59.1, 9.22)
- moved C4 2.33 mm to (66.6, 8.13)
- moved J2 2.32 mm to (37.8, 10.6)
- moved IC2 0.41 mm to (19.1, 25.6)
Connections:
- net GND: now also J3.3; no longer J3.1
- net P32: now also J3.1; no longer J3.3
Routing:
- net 3_3V: track 91.5 -> 97.9 mm
- net 3_3V_DIODE: track 66.2 -> 71.1 mm
- net P32: track 73.1 -> 76.0 mm
- net CAN_R: track 19.1 -> 17.6 mm
- net P00: track 50.3 -> 51.3 mm
- net P34: track 33.3 -> 34.1 mm
- net P35: track 32.7 -> 33.6 mm
- net P02: track 51.9 -> 52.8 mm
- net P27: track 52.3 -> 53.1 mm
- net P26: track 45.5 -> 46.2 mm
- net P36: track 48.6 -> 49.4 mm
- net P18: track 34.3 -> 33.6 mm
- net P25: track 45.3 -> 46.0 mm
- net P12: track 57.0 -> 57.7 mm
- net P14: track 52.8 -> 53.5 mm
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
Commit message: daily sync
Parts:
- removed J1: External, con-molex:6410-05
- removed J3: (no value), SparkFun-Connectors:1X03
- added F1: 0.75A 16V, fuses:1812L
- added J4: External, con-molex:6410-04
- moved D1 38.5 mm to (24.9, 49.1), flipped to the bottom
- moved C2 0.41 mm to (67.6, 16.1)
Connections:
- net P13 renamed SERVO1
- net P15 renamed SERVO2
- removed net 3_3V_DIODE: D1.C, IC2.14, J2.3, J2.4, J3.2
- removed net P12: IC2.2, X1.13
- new net N$4: F1.1, J4.4
- new net N$5: D1.C, IC2.14
- net 12V: now also F1.2; no longer J1.5
- net 5V: now also J2.3, J2.4
- net GND: now also J4.3, X1.13, X1.25; no longer J1.4, J3.3
- net LED: now also IC2.2; no longer J1.3
- net N$2: now also J4.1; no longer J1.1
- net N$3: now also J4.2; no longer J1.2
- net P32: no longer J3.1
Routing:
- net 3_3V_DIODE: track 71.1 -> 0.00 mm, vias 1 -> 0
- net P12: track 57.7 -> 0.00 mm
- net 5V: track 68.0 -> 123.0 mm
- net P32: track 76.0 -> 39.2 mm
- net 3_3V: track 97.9 -> 86.9 mm
- net N$4: track 0.00 -> 6.92 mm
- net LED: track 60.2 -> 54.6 mm
- net N$5: track 0.00 -> 5.05 mm
- net 12V: track 42.6 -> 44.5 mm
- net SERVO1: track 66.9 -> 67.9 mm
- net SERVO2: track 66.2 -> 67.1 mm
- net P22: track 22.8 -> 23.5 mm
- net P02: track 52.8 -> 53.4 mm
Other:
- board text added: "1 2"
- board text removed: "1 2 3"
- board text removed: "LED"
