File: data/Franks Flightsim Boards/Controler 3_5/Controler 3_5.sch (EAGLE design)
At the start: 19 parts, among them IC1 SN65HVD230, IC2 LOLIN32LITE, IC3 LD117AV33, IC4 7805T, J1 External, J2 FEMALE 2x3, X1 BUS

Commit message: Update dev status
Connections:
- net GND: now also J3.3; no longer J3.1
- net P32: now also J3.1; no longer J3.3
Changed lines of the file:
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@@
 <?xml version="1.0" encoding="utf-8"?>
 <!DOCTYPE eagle SYSTEM "eagle.dtd">
-<eagle version="8.7.0">
+<eagle version="9.0.0">
 <drawing>
 <settings>
@@
 <junction x="215.9" y="53.34"/>
 <wire x1="215.9" y1="53.34" x2="215.9" y2="45.72" width="0.1524" layer="91"/>
-<pinref part="J3" gate="J$1" pin="1"/>
-<wire x1="215.9" y1="45.72" x2="213.36" y2="45.72" width="0.1524" layer="91"/>
+<pinref part="J3" gate="J$1" pin="3"/>
+<wire x1="215.9" y1="45.72" x2="213.36" y2="40.64" width="0.1524" layer="91"/>
 </segment>
 <segment>
@@
 </segment>
 <segment>
-<pinref part="J3" gate="J$1" pin="3"/>
-<wire x1="213.36" y1="40.64" x2="218.44" y2="40.64" width="0.1524" layer="91"/>
+<pinref part="J3" gate="J$1" pin="1"/>
+<wire x1="213.36" y1="45.72" x2="218.44" y2="40.64" width="0.1524" layer="91"/>
 <label x="218.44" y="40.64" size="1.27" layer="95" xref="yes"/>
 </segment>

Commit message: daily sync
Parts:
- removed J1: External, con-molex:22-27-2051-05
- removed J3: (no value), SparkFun-Connectors:CONN_03
- added F1: 0.75A 16V, fuses:1812L
- added J4: External, con-molex:22-27-2041-04
Connections:
- net P13 renamed SERVO1
- net P15 renamed SERVO2
- removed net 3_3V_DIODE: D1.C, IC2.VCC, J2.3, J2.4, J3.2
- removed net P12: IC2.P12, X1-13.S
- new net N$4: F1.1, J4-4.S
- new net N$5: D1.C, IC2.VCC
- net 12V: now also F1.2; no longer J1-5.S
- net 5V: now also J2.3, J2.4
- net GND: now also J4-3.S, X1-13.S, X1-25.S; no longer J1-4.S, J3.3
- net LED: now also IC2.P12; no longer J1-3.S
- net N$2: now also J4-1.S; no longer J1-1.S
- net N$3: now also J4-2.S; no longer J1-2.S
- net P32: no longer J3.1
